Commit message: Complete jackal example running on Docker container

File: wild_visual_navigation_jackal/urdf/depth_camera.xacro (robot description, xacro)
@@ -41,4 +41,10 @@
             </inertial>
         </link>
+        <link name="optical_${name}_link"/>
+        <joint name="${name}_to_optical_${name}_link" type="fixed">
+            <origin xyz="0.0 0.0 0.0" rpy="${-90/180*pi} 0.0 ${-90/180*pi}" />
+            <parent link="${name}_link" />
+            <child link="optical_${name}_link" />
+        </joint>
         <gazebo reference="${name}_link">
             <turnGravityOff>true</turnGravityOff>
@@ -72,5 +78,5 @@
                     <depthImageInfoTopicName>/${name}/depth/camera_info</depthImageInfoTopicName>
                     <pointCloudTopicName>/${name}/depth/color/points</pointCloudTopicName>
-                    <frameName>${name}_link</frameName>
+                    <frameName>optical_${name}_link</frameName>
                     <pointCloudCutoff>0.105</pointCloudCutoff>
                     <pointCloudCutoffMax>8.0</pointCloudCutoffMax>
